Commit message: wheels

File: description/robot_core.xacro (robot description, xacro)
@@ -1,4 +1,5 @@
 <?xml version="1.0"?>
 <robot xmlns:xacro="http://www.ros.org/wiki/xacro">
+	 <xacro:include filename="inertial_macros.xacro"/>
          <material name = "white">
         	<color rgba = "1 1 1 1"/>
@@ -39,4 +40,90 @@
             		</geometry>
         	</collision>
-    	 </link>
+	</link>
+	<!-- left wheel -->
+    	<joint name = "left_wheel_joint" type="continuous">
+        	<parent link="base_link"/>
+        	<child link="left_wheel"/>
+        	<origin xyz="0.0 0.14 -0.07" rpy="-${pi/2} 0.0 0.0"/>
+        	<axis xyz="0.0 0.0 1"/>
+    	</joint>
+    	<link name="left_wheel">
+        	<visual>
+            		<origin xyz="0 0 0"/>
+            		<geometry>
+                		<cylinder radius="0.0325" length="0.026"/>
+            		</geometry>
+            		<material name="blue"/>
+        	</visual>
+        	<collision>
+            		<origin xyz="0 0 0"/>
+            		<geometry>
+                		<sphere radius="0.0325"/>
+            		</geometry>
+        	</collision>
+    	</link>
+    	<!-- right wheel -->
+    	<joint name = "right_wheel_joint" type="continuous">
+        	<parent link="base_link"/>
+        	<child link="right_wheel"/>
+        	<origin xyz="0.0 -0.14 -0.07" rpy="${pi/2} 0.0 0.0"/>
+        	<axis xyz="0.0 0.0 -1"/>
+    	</joint>
+    	<link name="right_wheel">
+        	<visual>
+            		<origin xyz="0 0 0"/>
+            		<geometry>
+                		<cylinder radius="0.0325" length="0.026"/>
+            		</geometry>
+            		<material name="blue"/>
+        	</visual>
+        	<collision>
+            		<origin xyz="0 0 0"/>
+            		<geometry>
+                		<sphere radius="0.0325"/>
+            		</geometry>
+        	</collision>
+    	</link>
+	<!-- front Castor wheel -->
+    	<joint name="front_castor_wheel_joint" type="fixed">
+        	<parent link="chassis"/>
+        	<child link="front_castor_wheel"/>
+        	<origin xyz="0.08 0.0 0.0" rpy="0.0 0.0 0.0"/>
+    	</joint>
+    	<link name="front_castor_wheel">
+        	<visual>
+            		<origin xyz="0 0 0"/>
+            		<geometry>
+                		<sphere radius="0.0325"/>
+            		</geometry>
+            		<material name="black"/>
+        	</visual>
+        	<collision>
+            		<origin xyz="0 0 0"/>
+            		<geometry>
+                		<sphere radius="0.0325"/>
+            		</geometry>
+        	</collision>
+    	</link>
+    	<!-- back Castor wheel -->
+    	<joint name="back_castor_wheel_joint" type="fixed">
+        	<parent link="chassis"/>
+        	<child link="back_castor_wheel"/>
+        	<origin xyz="-0.08 0.0 0.0" rpy="0.0 0.0 0.0"/>
+    	</joint>
+    	<link name="back_castor_wheel">
+        	<visual>
+            		<origin xyz="0 0 0"/>
+            		<geometry>
+                		<sphere radius="0.0325"/>
+            		</geometry>
+            		<material name="black"/>
+        	</visual>
+        	<collision>
+            		<origin xyz="0 0 0"/>
+            		<geometry>
+                		<sphere radius="0.0325"/>
+            		</geometry>
+        		</collision>
+    	</link>
 </robot>

Commit message: inertia

File: description/robot_core.xacro (robot description, xacro)
@@ -39,5 +39,8 @@
                 		<cylinder radius = "0.125" length = "0.07"/>
             		</geometry>
-        	</collision>
+		</collision>
+		<xacro:inertial_cylinder mass= "0.5" radius="0.125" length="0.07">
+            		<origin xyz="0.0 0.0 0.035" rpy="0.0 0.0 0.0"/>
+        	</xacro:inertial_cylinder>
 	</link>
 	<!-- left wheel -->
@@ -61,5 +64,8 @@
                 		<sphere radius="0.0325"/>
             		</geometry>
-        	</collision>
+		</collision>
+		<xacro:inertial_cylinder mass= "0.1" radius="0.0325" length="0.026">
+            		<origin xyz="0.0 0.0 0.0" rpy="0.0 0.0 0.0"/>
+          	</xacro:inertial_cylinder>
     	</link>
     	<!-- right wheel -->
@@ -83,5 +89,8 @@
                 		<sphere radius="0.0325"/>
             		</geometry>
-        	</collision>
+		</collision>
+		 <xacro:inertial_cylinder mass= "0.1" radius="0.0325" length="0.026">
+            		<origin xyz="0.0 0.0 0.0" rpy="0.0 0.0 0.0"/>
+        	</xacro:inertial_cylinder>
     	</link>
 	<!-- front Castor wheel -->
@@ -104,5 +113,8 @@
                 		<sphere radius="0.0325"/>
             		</geometry>
-        	</collision>
+		</collision>
+		<xacro:inertial_sphere mass= "0.1" radius="0.0325">
+            		<origin xyz="0.0 0.0 0.0" rpy="0.0 0.0 0.0"/>
+        	</xacro:inertial_sphere>
     	</link>
     	<!-- back Castor wheel -->
@@ -125,5 +137,8 @@
                 		<sphere radius="0.0325"/>
             		</geometry>
-        		</collision>
+        	</collision>
+		<xacro:inertial_sphere mass= "0.1" radius="0.0325">
+            		<origin xyz="0.0 0.0 0.0" rpy="0.0 0.0 0.0"/>
+        	</xacro:inertial_sphere>
     	</link>
 </robot>
