Commit message: driver

File: description/robot.urdf.xacro (robot description, xacro)
@@ -2,3 +2,4 @@
 <robot xmlns:xacro="http://www.ros.org/wiki/xacro"  name="robot">
 	<xacro:include filename="robot_core.xacro" />
+	<xacro:include filename="gazebo_control.xacro" />
 </robot>

File: description/robot_core.xacro (robot description, xacro)
@@ -44,4 +44,7 @@
         	</xacro:inertial_cylinder>
 	</link>
+	<gazebo reference="chassis">
+        	<material>Gazebo/White</material>
+    	</gazebo>
 	<!-- left wheel -->
     	<joint name = "left_wheel_joint" type="continuous">
@@ -68,5 +71,8 @@
             		<origin xyz="0.0 0.0 0.0" rpy="0.0 0.0 0.0"/>
           	</xacro:inertial_cylinder>
-    	</link>
+	</link>
+	<gazebo reference="left_wheel">
+        	<material>Gazebo/Blue</material>
+    	</gazebo>
     	<!-- right wheel -->
     	<joint name = "right_wheel_joint" type="continuous">
@@ -93,5 +99,8 @@
             		<origin xyz="0.0 0.0 0.0" rpy="0.0 0.0 0.0"/>
         	</xacro:inertial_cylinder>
-    	</link>
+	</link>
+	<gazebo reference="right_wheel">
+        	<material>Gazebo/Blue</material>
+    	</gazebo>
 	<!-- front Castor wheel -->
     	<joint name="front_castor_wheel_joint" type="fixed">
@@ -117,5 +126,10 @@
             		<origin xyz="0.0 0.0 0.0" rpy="0.0 0.0 0.0"/>
         	</xacro:inertial_sphere>
-    	</link>
+	</link>
+	<gazebo reference="front_castor_wheel">
+        	<material>Gazebo/Black</material>
+        	<mu1 value="0.001"/>
+        	<mu2 value="0.001"/>
+    	</gazebo>
     	<!-- back Castor wheel -->
     	<joint name="back_castor_wheel_joint" type="fixed">
@@ -141,4 +155,9 @@
             		<origin xyz="0.0 0.0 0.0" rpy="0.0 0.0 0.0"/>
         	</xacro:inertial_sphere>
-    	</link>
+	</link>
+	<gazebo reference="back_castor_wheel">
+        	<material>Gazebo/Black</material>
+        	<mu1 value="0.001"/>
+        	<mu2 value="0.001"/>
+	</gazebo>
 </robot>
